Commit message: Day 26: Add visual geometry and materials to MIGRO URDF

File: 06_urdf/migro_description/urdf/migro.urdf (robot description, URDF)
Before this commit: robot migro, 2 links, 1 joints
Links:
- link base_link: geometry visual box size=0.5 0.4 0.2
- link camera_link: geometry visual box size=0.08 0.08 0.05
