Commit message: Day 30: Build four-wheel MIGRO robot and document progress

File: migro_description/urdf/migro.urdf (robot description, URDF)
Before this commit: robot migro, 2 links, 1 joints
Links:
- added link left_front_wheel; visual cylinder length=0.03 radius=0.05
- added link left_rear_wheel; visual cylinder length=0.03 radius=0.05
- added link right_front_wheel; visual cylinder length=0.03 radius=0.05
- added link right_rear_wheel; visual cylinder length=0.03 radius=0.05
Joints:
- added joint left_front_wheel_joint: type fixed, parent base_link, child left_front_wheel, origin xyz=0.18 0.20 0.05 rpy=1.5708 0 0
- added joint left_rear_wheel_joint: type fixed, parent base_link, child left_rear_wheel, origin xyz=-0.18 0.20 0.05 rpy=1.5708 0 0
- added joint right_front_wheel_joint: type fixed, parent base_link, child right_front_wheel, origin xyz=0.18 -0.20 0.05 rpy=1.5708 0 0
- added joint right_rear_wheel_joint: type fixed, parent base_link, child right_rear_wheel, origin xyz=-0.18 -0.20 0.05 rpy=1.5708 0 0
