Commit message: Complete MIGRO differential drive control

File: migro_description/urdf/macros.xacro (robot description, xacro)
@@ -44,5 +44,5 @@
           rpy="1.5708 0 0"/>
       <!-- Wheel rotates about its local Y-axis -->
-      <axis xyz="0 1 0"/>
+      <axis xyz="0 0 -1"/>
     </joint>
   </xacro:macro>
