Commit message: Day 33: Improve Xacro with parametric chassis elevation

File: migro_description/urdf/migro.urdf.xacro (robot description, xacro)
@@ -1,7 +1,35 @@
 <?xml version="1.0"?>
-<robot
-    xmlns:xacro="http://www.ros.org/wiki/xacro"
-    name="migro">
-  <!-- ================= Materials ================= -->
+<robot xmlns:xacro="http://www.ros.org/wiki/xacro" name="migro">
+  <!-- ========================================================= -->
+  <!-- Robot Properties -->
+  <!-- ========================================================= -->
+  <!-- Chassis -->
+  <xacro:property name="chassis_length" value="0.5"/>
+  <xacro:property name="chassis_width" value="0.4"/>
+  <xacro:property name="chassis_height" value="0.2"/>
+  <!-- Wheels -->
+  <xacro:property name="wheel_radius" value="0.10"/>
+  <xacro:property name="wheel_width" value="0.06"/>
+  <xacro:property name="wheel_x" value="0.18"/>
+  <xacro:property name="wheel_y" value="0.24"/>
+  <xacro:property name="wheel_z" value="${wheel_radius}"/>
+  <!-- Ground Clearance -->
+  <xacro:property name="ground_clearance" value="0.05"/>
+  <!-- Height of chassis above the world -->
+  <xacro:property
+      name="body_z"
+      value="${wheel_radius + ground_clearance + chassis_height/2}"/>
+  <!-- Camera -->
+  <xacro:property name="camera_length" value="0.08"/>
+  <xacro:property name="camera_width" value="0.08"/>
+  <xacro:property name="camera_height" value="0.05"/>
+  <xacro:property name="camera_x" value="0.0"/>
+  <xacro:property name="camera_y" value="0.0"/>
+  <xacro:property
+      name="camera_z"
+      value="${body_z + chassis_height/2 - 0.05}"/>
+  <!-- ========================================================= -->
+  <!-- Materials -->
+  <!-- ========================================================= -->
   <material name="blue">
     <color rgba="0 0 1 1"/>
@@ -13,85 +41,100 @@
     <color rgba="0.5 0.5 0.5 1"/>
   </material>
-  <!-- ================= Chassis ================= -->
+  <!-- ========================================================= -->
+  <!-- Chassis -->
+  <!-- ========================================================= -->
   <link name="base_link">
     <visual>
-      <origin xyz="0 0 0.1"/>
+      <origin xyz="0 0 ${body_z}"/>
       <geometry>
-        <box size="0.5 0.4 0.2"/>
+        <box size="${chassis_length} ${chassis_width} ${chassis_height}"/>
       </geometry>
       <material name="blue"/>
     </visual>
+    <collision>
+      <origin xyz="0 0 ${body_z}"/>
+      <geometry>
+        <box size="${chassis_length} ${chassis_width} ${chassis_height}"/>
+      </geometry>
+    </collision>
   </link>
-  <!-- ================= Camera ================= -->
+  <!-- ========================================================= -->
+  <!-- Camera -->
+  <!-- ========================================================= -->
   <link name="camera_link">
     <visual>
-      <origin xyz="0 0 0.025"/>
+      <origin xyz="0 0 ${camera_height/2}"/>
       <geometry>
-        <box size="0.08 0.08 0.05"/>
+        <box size="${camera_length} ${camera_width} ${camera_height}"/>
       </geometry>
       <material name="black"/>
     </visual>
+    <collision>
+      <origin xyz="0 0 ${camera_height/2}"/>
+      <geometry>
+        <box size="${camera_length} ${camera_width} ${camera_height}"/>
+      </geometry>
+    </collision>
   </link>
   <joint name="camera_joint" type="fixed">
     <parent link="base_link"/>
     <child link="camera_link"/>
-    <origin xyz="0 0 0.15" rpy="0 0 0"/>
+    <origin xyz="${camera_x} ${camera_y} ${camera_z}" rpy="0 0 0"/>
   </joint>
-  <!-- ================= Left Front Wheel ================= -->
-  <link name="left_front_wheel">
-    <visual>
-      <origin xyz="0 0 0"/>
-      <geometry>
-        <cylinder radius="0.05" length="0.03"/>
-      </geometry>
-      <material name="grey"/>
-    </visual>
-  </link>
-  <joint name="left_front_wheel_joint" type="fixed">
+  <!-- ========================================================= -->
+  <!-- Wheel Macro -->
+  <!-- ========================================================= -->
+  <xacro:macro name="wheel" params="name x y z">
+    <link name="${name}">
+      <visual>
+        <origin xyz="0 0 0"/>
+        <geometry>
+          <cylinder
+              radius="${wheel_radius}"
+              length="${wheel_width}"/>
+        </geometry>
+        <material name="grey"/>
+      </visual>
+      <collision>
+        <origin xyz="0 0 0"/>
+        <geometry>
+          <cylinder
+              radius="${wheel_radius}"
+              length="${wheel_width}"/>
+        </geometry>
+      </collision>
+    </link>
+    <joint
+        name="${name}_joint"
+        type="fixed">
       <parent link="base_link"/>
-      <child link="left_front_wheel"/>
-      <origin xyz="0.18 0.20 0.05" rpy="1.5708 0 0"/>
-  </joint>
-  <!-- ================= Right Front Wheel ================= -->
-  <link name="right_front_wheel">
-    <visual>
-      <geometry>
-        <cylinder radius="0.05" length="0.03"/>
-      </geometry>
-      <material name="grey"/>
-    </visual>
-  </link>
-  <joint name="right_front_wheel_joint" type="fixed">
-      <parent link="base_link"/>
-      <child link="right_front_wheel"/>
-      <origin xyz="0.18 -0.20 0.05" rpy="1.5708 0 0"/>
-  </joint>
-  <!-- ================= Left Rear Wheel ================= -->
-  <link name="left_rear_wheel">
-    <visual>
-      <geometry>
-        <cylinder radius="0.05" length="0.03"/>
-      </geometry>
-      <material name="grey"/>
-    </visual>
-  </link>
-  <joint name="left_rear_wheel_joint" type="fixed">
-      <parent link="base_link"/>
-      <child link="left_rear_wheel"/>
-      <origin xyz="-0.18 0.20 0.05" rpy="1.5708 0 0"/>
-  </joint>
-  <!-- ================= Right Rear Wheel ================= -->
-  <link name="right_rear_wheel">
-    <visual>
-      <geometry>
-        <cylinder radius="0.05" length="0.03"/>
-      </geometry>
-      <material name="grey"/>
-    </visual>
-  </link>
-  <joint name="right_rear_wheel_joint" type="fixed">
-      <parent link="base_link"/>
-      <child link="right_rear_wheel"/>
-      <origin xyz="-0.18 -0.20 0.05" rpy="1.5708 0 0"/>
-  </joint>
+      <child link="${name}"/>
+      <origin
+          xyz="${x} ${y} ${z}"
+          rpy="1.5708 0 0"/>
+    </joint>
+  </xacro:macro>
+  <!-- ========================================================= -->
+  <!-- Wheels -->
+  <!-- ========================================================= -->
+  <xacro:wheel
+      name="left_front_wheel"
+      x="${wheel_x}"
+      y="${wheel_y}"
+      z="${wheel_z}"/>
+  <xacro:wheel
+      name="right_front_wheel"
+      x="${wheel_x}"
+      y="${-wheel_y}"
+      z="${wheel_z}"/>
+  <xacro:wheel
+      name="left_rear_wheel"
+      x="${-wheel_x}"
+      y="${wheel_y}"
+      z="${wheel_z}"/>
+  <xacro:wheel
+      name="right_rear_wheel"
+      x="${-wheel_x}"
+      y="${-wheel_y}"
+      z="${wheel_z}"/>
 </robot>

Commit message: Day 34: Modularize MIGRO robot description

File: migro_description/urdf/migro.urdf.xacro (robot description, xacro)
@@ -2,139 +2,10 @@
 <robot xmlns:xacro="http://www.ros.org/wiki/xacro" name="migro">
   <!-- ========================================================= -->
-  <!-- Robot Properties -->
+  <!-- Includes -->
   <!-- ========================================================= -->
-  <!-- Chassis -->
-  <xacro:property name="chassis_length" value="0.5"/>
-  <xacro:property name="chassis_width" value="0.4"/>
-  <xacro:property name="chassis_height" value="0.2"/>
-  <!-- Wheels -->
-  <xacro:property name="wheel_radius" value="0.10"/>
-  <xacro:property name="wheel_width" value="0.06"/>
-  <xacro:property name="wheel_x" value="0.18"/>
-  <xacro:property name="wheel_y" value="0.24"/>
-  <xacro:property name="wheel_z" value="${wheel_radius}"/>
-  <!-- Ground Clearance -->
-  <xacro:property name="ground_clearance" value="0.05"/>
-  <!-- Height of chassis above the world -->
-  <xacro:property
-      name="body_z"
-      value="${wheel_radius + ground_clearance + chassis_height/2}"/>
-  <!-- Camera -->
-  <xacro:property name="camera_length" value="0.08"/>
-  <xacro:property name="camera_width" value="0.08"/>
-  <xacro:property name="camera_height" value="0.05"/>
-  <xacro:property name="camera_x" value="0.0"/>
-  <xacro:property name="camera_y" value="0.0"/>
-  <xacro:property
-      name="camera_z"
-      value="${body_z + chassis_height/2 - 0.05}"/>
-  <!-- ========================================================= -->
-  <!-- Materials -->
-  <!-- ========================================================= -->
-  <material name="blue">
-    <color rgba="0 0 1 1"/>
-  </material>
-  <material name="black">
-    <color rgba="0.1 0.1 0.1 1"/>
-  </material>
-  <material name="grey">
-    <color rgba="0.5 0.5 0.5 1"/>
-  </material>
-  <!-- ========================================================= -->
-  <!-- Chassis -->
-  <!-- ========================================================= -->
-  <link name="base_link">
-    <visual>
-      <origin xyz="0 0 ${body_z}"/>
-      <geometry>
-        <box size="${chassis_length} ${chassis_width} ${chassis_height}"/>
-      </geometry>
-      <material name="blue"/>
-    </visual>
-    <collision>
-      <origin xyz="0 0 ${body_z}"/>
-      <geometry>
-        <box size="${chassis_length} ${chassis_width} ${chassis_height}"/>
-      </geometry>
-    </collision>
-  </link>
-  <!-- ========================================================= -->
-  <!-- Camera -->
-  <!-- ========================================================= -->
-  <link name="camera_link">
-    <visual>
-      <origin xyz="0 0 ${camera_height/2}"/>
-      <geometry>
-        <box size="${camera_length} ${camera_width} ${camera_height}"/>
-      </geometry>
-      <material name="black"/>
-    </visual>
-    <collision>
-      <origin xyz="0 0 ${camera_height/2}"/>
-      <geometry>
-        <box size="${camera_length} ${camera_width} ${camera_height}"/>
-      </geometry>
-    </collision>
-  </link>
-  <joint name="camera_joint" type="fixed">
-    <parent link="base_link"/>
-    <child link="camera_link"/>
-    <origin xyz="${camera_x} ${camera_y} ${camera_z}" rpy="0 0 0"/>
-  </joint>
-  <!-- ========================================================= -->
-  <!-- Wheel Macro -->
-  <!-- ========================================================= -->
-  <xacro:macro name="wheel" params="name x y z">
-    <link name="${name}">
-      <visual>
-        <origin xyz="0 0 0"/>
-        <geometry>
-          <cylinder
-              radius="${wheel_radius}"
-              length="${wheel_width}"/>
-        </geometry>
-        <material name="grey"/>
-      </visual>
-      <collision>
-        <origin xyz="0 0 0"/>
-        <geometry>
-          <cylinder
-              radius="${wheel_radius}"
-              length="${wheel_width}"/>
-        </geometry>
-      </collision>
-    </link>
-    <joint
-        name="${name}_joint"
-        type="fixed">
-      <parent link="base_link"/>
-      <child link="${name}"/>
-      <origin
-          xyz="${x} ${y} ${z}"
-          rpy="1.5708 0 0"/>
-    </joint>
-  </xacro:macro>
-  <!-- ========================================================= -->
-  <!-- Wheels -->
-  <!-- ========================================================= -->
-  <xacro:wheel
-      name="left_front_wheel"
-      x="${wheel_x}"
-      y="${wheel_y}"
-      z="${wheel_z}"/>
-  <xacro:wheel
-      name="right_front_wheel"
-      x="${wheel_x}"
-      y="${-wheel_y}"
-      z="${wheel_z}"/>
-  <xacro:wheel
-      name="left_rear_wheel"
-      x="${-wheel_x}"
-      y="${wheel_y}"
-      z="${wheel_z}"/>
-  <xacro:wheel
-      name="right_rear_wheel"
-      x="${-wheel_x}"
-      y="${-wheel_y}"
-      z="${wheel_z}"/>
+  <xacro:include filename="properties.xacro"/>
+  <xacro:include filename="materials.xacro"/>
+  <xacro:include filename="chassis.xacro"/>
+  <xacro:include filename="camera.xacro"/>
+  <xacro:include filename="macros.xacro"/>  <!-- ========================================================= -->  <!-- Wheels -->  <!-- ========================================================= -->  <xacro:wheel      name="left_front_wheel"      x="${wheel_x}"      y="${wheel_y}"      z="${wheel_z}"/>  <xacro:wheel      name="right_front_wheel"      x="${wheel_x}"      y="${-wheel_y}"      z="${wheel_z}"/>  <xacro:wheel      name="left_rear_wheel"      x="${-wheel_x}"      y="${wheel_y}"      z="${wheel_z}"/>  <xacro:wheel      name="right_rear_wheel"      x="${-wheel_x}"      y="${-wheel_y}"      z="${wheel_z}"/>
 </robot>

Commit message: Add 2D LIDAR sensor with Gazebo Sim integration
- New lidar.xacro: physical mount + gpu_lidar sensor definition
- Add missing Sensors system plugin to world file (root cause of
  sensor data not publishing)
- Bridge /scan topic via ros_gz_bridge
- Fix sensor frame_id using gz_frame_id (not frame_id) so /scan
  resolves correctly against the URDF-based TF tree
- Verified against known obstacle: measured range matches expected
  geometry within display precision

File: migro_description/urdf/migro.urdf.xacro (robot description, xacro)
@@ -8,4 +8,5 @@
   <xacro:include filename="chassis.xacro"/>
   <xacro:include filename="camera.xacro"/>
+  <xacro:include filename="lidar.xacro"/>
   <xacro:include filename="macros.xacro"/>
   <xacro:include filename="ros2_control.xacro"/>

File: migro_description/urdf/properties.xacro (robot description, xacro)
@@ -29,3 +29,11 @@
       name="camera_z"
       value="${body_z + chassis_height/2 - 0.05}"/>
+  <!-- LIDAR -->
+  <xacro:property name="lidar_radius" value="0.04"/>
+  <xacro:property name="lidar_height" value="0.05"/>
+  <xacro:property name="lidar_x" value="${chassis_length/2 - 0.05}"/>
+  <xacro:property name="lidar_y" value="0.0"/>
+  <xacro:property
+     name="lidar_z"
+     value="${body_z + chassis_height/2 + lidar_height/2}"/>
 </robot>
