Commit message: debug Gazebo simulation issues

File: migro_description/urdf/camera.xacro (robot description, xacro)
@@ -18,4 +18,15 @@
       </geometry>
     </collision>
+    <inertial>
+      <origin xyz="0 0 0.025" rpy="0 0 0"/>
+      <mass value="0.2"/>
+      <inertia
+          ixx="0.0001"
+          ixy="0.0"
+          ixz="0.0"
+          iyy="0.0001"
+          iyz="0.0"
+          izz="0.0001"/>
+    </inertial>
   </link>
   <joint name="camera_joint" type="fixed">

File: migro_description/urdf/chassis.xacro (robot description, xacro)
@@ -5,4 +5,15 @@
   <!-- ========================================================= -->
   <link name="base_link">
+    <inertial>
+     <origin xyz="0 0 ${body_z}" rpy="0 0 0"/>
+     <mass value="5.0"/>
+     <inertia
+      ixx="0.08"
+      ixy="0.0"
+      ixz="0.0"
+      iyy="0.12"
+      iyz="0.0"
+      izz="0.15"/>
+    </inertial>
     <visual>
       <origin xyz="0 0 ${body_z}"/>

File: migro_description/urdf/macros.xacro (robot description, xacro)
@@ -23,8 +23,19 @@
         </geometry>
       </collision>
+      <inertial>
+        <origin xyz="0 0 0"/>
+        <mass value="0.5"/>
+        <inertia
+            ixx="0.001"
+            ixy="0.0"
+            ixz="0.0"
+            iyy="0.001"
+            iyz="0.0"
+            izz="0.001"/>
+      </inertial>
     </link>
     <joint
         name="${name}_joint"
-        type="fixed">
+        type="continuous">
       <parent link="base_link"/>
       <child link="${name}"/>
@@ -32,4 +43,6 @@
           xyz="${x} ${y} ${z}"
           rpy="1.5708 0 0"/>
+      <!-- Wheel rotates about its local Y-axis -->
+      <axis xyz="0 1 0"/>
     </joint>
   </xacro:macro>

File: migro_description/urdf/migro.urdf.xacro (robot description, xacro)
@@ -8,4 +8,26 @@
   <xacro:include filename="chassis.xacro"/>
   <xacro:include filename="camera.xacro"/>
-  <xacro:include filename="macros.xacro"/>  <!-- ========================================================= -->  <!-- Wheels -->  <!-- ========================================================= -->  <xacro:wheel      name="left_front_wheel"      x="${wheel_x}"      y="${wheel_y}"      z="${wheel_z}"/>  <xacro:wheel      name="right_front_wheel"      x="${wheel_x}"      y="${-wheel_y}"      z="${wheel_z}"/>  <xacro:wheel      name="left_rear_wheel"      x="${-wheel_x}"      y="${wheel_y}"      z="${wheel_z}"/>  <xacro:wheel      name="right_rear_wheel"      x="${-wheel_x}"      y="${-wheel_y}"      z="${wheel_z}"/>
+  <xacro:include filename="macros.xacro"/>
+  <xacro:include filename="ros2_control.xacro"/>
+   <!-- =================== -->  <!-- Wheels -->  <!-- ========================== -->
+   <xacro:wheel
+    name="left_front_wheel"
+    x="${wheel_x}"
+    y="${wheel_y}"
+    z="${wheel_z}"/>
+<xacro:wheel
+    name="right_front_wheel"
+    x="${wheel_x}"
+    y="${-wheel_y}"
+    z="${wheel_z}"/>
+<xacro:wheel
+    name="left_rear_wheel"
+    x="${-wheel_x}"
+    y="${wheel_y}"
+    z="${wheel_z}"/>
+<xacro:wheel
+    name="right_rear_wheel"
+    x="${-wheel_x}"
+    y="${-wheel_y}"
+    z="${wheel_z}"/>
 </robot>

Commit message: Day 60: add camera sensor with gz-sim optical_frame_id fix
- camera link/joint, optical frame, gz-sim camera sensor
- ros_gz_bridge for image_raw + camera_info
- camera_viewer.py cv_bridge subscriber
- world lighting/materials, LiDAR/camera clearance fix
- root cause: sensor must attach to unrotated link + optical_frame_id

File: migro_description/urdf/camera.xacro (robot description, xacro)
@@ -35,3 +35,32 @@
     <origin xyz="${camera_x} ${camera_y} ${camera_z}" rpy="0 0 0"/>
   </joint>
+    <!-- Optical frame: rotates from URDF convention (x-forward, z-up)
+       to camera/ROS convention (z-forward, x-right, y-down) -->
+  <link name="camera_link_optical"/>
+  <joint name="camera_optical_joint" type="fixed">
+    <parent link="camera_link"/>
+    <child link="camera_link_optical"/>
+    <origin xyz="${camera_length/2 + 0.01} 0 ${camera_height/2}" rpy="${-pi/2} 0 ${-pi/2}"/>
+  </joint>
+ <gazebo reference="camera_link">
+  <sensor name="camera_sensor" type="camera">
+    <always_on>true</always_on>
+    <update_rate>30</update_rate>
+    <visualize>true</visualize>
+    <topic>camera/image_raw</topic>
+    <camera>
+      <horizontal_fov>1.089</horizontal_fov>
+      <image>
+        <width>640</width>
+        <height>480</height>
+        <format>R8G8B8</format>
+      </image>
+      <clip>
+        <near>0.05</near>
+        <far>10.0</far>
+      </clip>
+      <optical_frame_id>camera_link_optical</optical_frame_id>
+    </camera>
+  </sensor>
+ </gazebo>
 </robot>

File: migro_description/urdf/properties.xacro (robot description, xacro)
@@ -20,13 +20,4 @@
       name="body_z"
       value="${wheel_radius + ground_clearance + chassis_height/2}"/>
-  <!-- Camera -->
-  <xacro:property name="camera_length" value="0.08"/>
-  <xacro:property name="camera_width" value="0.08"/>
-  <xacro:property name="camera_height" value="0.05"/>
-  <xacro:property name="camera_x" value="0.0"/>
-  <xacro:property name="camera_y" value="0.0"/>
-  <xacro:property
-      name="camera_z"
-      value="${body_z + chassis_height/2 - 0.05}"/>
   <!-- LIDAR -->
   <xacro:property name="lidar_radius" value="0.04"/>
@@ -37,3 +28,12 @@
      name="lidar_z"
      value="${body_z + chassis_height/2 + lidar_height/2}"/>
+  <!-- Camera -->
+  <xacro:property name="camera_length" value="0.08"/>
+  <xacro:property name="camera_width" value="0.08"/>
+  <xacro:property name="camera_height" value="0.05"/>
+  <xacro:property name="camera_x" value="${chassis_length/2 + camera_length/2}"/>
+  <xacro:property name="camera_y" value="0.0"/>
+  <xacro:property
+      name="camera_z"
+      value="${lidar_z - lidar_height/2 - camera_height/2 - 0.03}"/>
 </robot>
